File: gbc-cm4-aio.kicad_sch (KiCad schematic)
At the start: 131 parts, among them J1 Conn_01x40, J2 AudioJack2_Ground_Switch, J4 DM3D-SF, J6 Conn_01x11, J7 Conn_01x02, P1 USB_C_Plug_USB2.0, Q1 2N7002E, Q1 AO4407C, SW1 SW_Push, SW2 BOOT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

Commit message: minor tweaks
Parts:
- added VBAT1: VBAT, TestPoint:TestPoint_Pad_D1.0mm, symbol Connector:TestPoint
- added VBUS1: VBUS, TestPoint:TestPoint_Pad_D1.0mm, symbol Connector:TestPoint
- added VIN1: VIN, TestPoint:TestPoint_Pad_D1.0mm, symbol Connector:TestPoint
- C1, C2: footprint PintryParts-Footprints:C_0402_1005Metric -> PintryParts-Footprints:C_0603_1608Metric; Size 0402 -> 0603
- R1, R2, R34: footprint Capacitor_SMD:C_0603_1608Metric -> Resistor_SMD:R_0603_1608Metric
Connections:
- net VBAT: now also VBAT1.1
- net VBUS: now also VBUS1.1
- net VIN: now also VIN1.1
Changed lines of the file:
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@@
   (junction (at 116.205 86.36) (diameter 0) (color 0 0 0 0)
   )
+  (junction (at 542.29 206.375) (diameter 0) (color 0 0 0 0)
+  )
   (junction (at 417.195 238.76) (diameter 0) (color 0 0 0 0)
   )
@@
     (stroke (width 0) (type default))
   )
+  (wire (pts (xy 540.385 206.375) (xy 542.29 206.375))
+    (stroke (width 0) (type default))
+  )
   (wire (pts (xy 485.14 253.365) (xy 485.14 250.19))
     (stroke (width 0) (type default))
@@
     (stroke (width 0) (type default))
   )
+  (wire (pts (xy 492.76 210.82) (xy 492.76 213.36))
+    (stroke (width 0) (type default))
+  )
   (wire (pts (xy 111.125 306.07) (xy 127.635 306.07))
     (stroke (width 0) (type default))
@@
     (stroke (width 0) (type default))
   )
+  (wire (pts (xy 475.615 126.365) (xy 475.615 128.27))
+    (stroke (width 0) (type default))
+  )
   (wire (pts (xy 73.66 98.425) (xy 73.66 107.315))
     (stroke (width 0) (type default))
@@
       (effects (font (size 1.27 1.27)) (justify left))
     )
-    (property "Footprint" "PintryParts-Footprints:C_0402_1005Metric" (at 154.305 323.85 0)
+    (property "Footprint" "PintryParts-Footprints:C_0603_1608Metric" (at 154.305 323.85 0)
       (effects (font (size 1.27 1.27)) hide)
     )
@@
       (effects (font (size 1.27 1.27)) (justify left))
     )
-    (property "Size" "0402" (at 156.337 325.882 0)
+    (property "Size" "0603" (at 156.337 325.882 0)
       (effects (font (size 1.27 1.27)) (justify left))
     )
@@
       (effects (font (size 1.27 1.27)) (justify left))
     )
-    (property "Footprint" "Capacitor_SMD:C_0603_1608Metric" (at 366.141 216.916 90)
+    (property "Footprint" "Resistor_SMD:R_0603_1608Metric" (at 366.141 216.916 90)
       (effects (font (size 1.27 1.27)) hide)
     )
@@
     )
   )
+  (symbol (lib_id "Connector:TestPoint") (at 540.385 206.375 90) (unit 1)
+    (in_bom yes) (on_board yes) (dnp no)
+    (property "Reference" "VBUS1" (at 532.8284 208.28 0)
+      (effects (font (size 1.27 1.27)) (justify left))
+    )
+    (property "Value" "VBUS" (at 534.7334 208.28 0)
+      (effects (font (size 1.27 1.27)) (justify left))
+    )
+    (property "Footprint" "TestPoint:TestPoint_Pad_D1.0mm" (at 540.385 201.295 0)
+      (effects (font (size 1.27 1.27)) hide)
+    )
+    (property "Datasheet" "~" (at 540.385 201.295 0)
+      (effects (font (size 1.27 1.27)) hide)
+    )
+    (pin "1")
+    (instances
+      (project "gbc-cm4-aio"
+        (path "/4dda0f32-68f6-467e-9c4a-af7e2b8a8793"
+          (reference "VBUS1") (unit 1)
+        )
+      )
+    )
+  )
   (symbol (lib_id "power:GND") (at 321.945 245.745 0) (unit 1)
     (in_bom yes) (on_board yes) (dnp no) (fields_autoplaced)
@@
     )
   )
+  (symbol (lib_id "Connector:TestPoint") (at 475.615 126.365 0) (unit 1)
+    (in_bom yes) (on_board yes) (dnp no)
+    (property "Reference" "VIN1" (at 473.71 118.8084 0)
+      (effects (font (size 1.27 1.27)) (justify left))
+    )
+    (property "Value" "VIN" (at 473.71 120.7134 0)
+      (effects (font (size 1.27 1.27)) (justify left))
+    )
+    (property "Footprint" "TestPoint:TestPoint_Pad_D1.0mm" (at 480.695 126.365 0)
+      (effects (font (size 1.27 1.27)) hide)
+    )
+    (property "Datasheet" "~" (at 480.695 126.365 0)
+      (effects (font (size 1.27 1.27)) hide)
+    )
+    (pin "1")
+    (instances
+      (project "gbc-cm4-aio"
+        (path "/4dda0f32-68f6-467e-9c4a-af7e2b8a8793"
+          (reference "VIN1") (unit 1)
+        )
+      )
+    )
+  )
   (symbol (lib_id "power:-5V") (at 76.835 57.15 0) (unit 1)
     (in_bom yes) (on_board yes) (dnp no) (fields_autoplaced)
@@
     )
   )
+  (symbol (lib_id "Connector:TestPoint") (at 492.76 210.82 0) (unit 1)
+    (in_bom yes) (on_board yes) (dnp no)
+    (property "Reference" "VBAT1" (at 490.855 203.2634 0)
+      (effects (font (size 1.27 1.27)) (justify left))
+    )
+    (property "Value" "VBAT" (at 490.855 205.1684 0)
+      (effects (font (size 1.27 1.27)) (justify left))
+    )
+    (property "Footprint" "TestPoint:TestPoint_Pad_D1.0mm" (at 497.84 210.82 0)
+      (effects (font (size 1.27 1.27)) hide)
+    )
+    (property "Datasheet" "~" (at 497.84 210.82 0)
+      (effects (font (size 1.27 1.27)) hide)
+    )
+    (pin "1")
+    (instances
+      (project "gbc-cm4-aio"
+        (path "/4dda0f32-68f6-467e-9c4a-af7e2b8a8793"
+          (reference "VBAT1") (unit 1)
+        )
+      )
+    )
+  )
   (symbol (lib_id "power:GND") (at 356.87 76.2 0) (unit 1)
     (in_bom yes) (on_board yes) (dnp no)
@@
       (effects (font (size 1.27 1.27)) (justify left))
     )
-    (property "Footprint" "Capacitor_SMD:C_0603_1608Metric" (at 223.774 68.834 90)
+    (property "Footprint" "Resistor_SMD:R_0603_1608Metric" (at 223.774 68.834 90)
       (effects (font (size 1.27 1.27)) hide)
     )
@@
       (effects (font (size 1.27 1.27)) (justify left))
     )
-    (property "Footprint" "Capacitor_SMD:C_0603_1608Metric" (at 223.774 51.054 90)
+    (property "Footprint" "Resistor_SMD:R_0603_1608Metric" (at 223.774 51.054 90)
       (effects (font (size 1.27 1.27)) hide)
     )
@@
       (effects (font (size 1.27 1.27)) (justify left))
     )
-    (property "Footprint" "PintryParts-Footprints:C_0402_1005Metric" (at 164.465 323.85 0)
+    (property "Footprint" "PintryParts-Footprints:C_0603_1608Metric" (at 164.465 323.85 0)
       (effects (font (size 1.27 1.27)) hide)
     )
@@
       (effects (font (size 1.27 1.27)) (justify left))
     )
-    (property "Size" "0402" (at 166.497 325.882 0)
+    (property "Size" "0603" (at 166.497 325.882 0)
       (effects (font (size 1.27 1.27)) (justify left))
     )

Commit message: MAX17048 package fix, added front power led, minor tweaks
Parts:
- added D11: APA2107SECK, LED_SMD:LED_0603_1608Metric, symbol PintryParts-Symbols:APA2107SECK
- added R42: 1K, Resistor_SMD:R_0603_1608Metric, symbol Device:R_US
- U4: footprint Package_DFN_QFN:TDFN-14-1EP_3x3mm_P0.4mm_EP1.78x2.35mm -> Package_DFN_QFN:TDFN-8-1EP_2x2mm_P0.5mm_EP0.8x1.2mm
Connections:
- net +3V3: now also D11.2 (A)
- net GND: now also R42.2
- new net: D11.1 (K), R42.1
Changed lines of the file:
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@@
   (no_connect (at 254.635 240.03))
   (no_connect (at 50.165 298.45))
+  (wire (pts (xy 174.625 104.14) (xy 182.245 104.14))
+    (stroke (width 0) (type solid))
+  )
   (wire (pts (xy 191.135 295.91) (xy 193.675 295.91))
     (stroke (width 0) (type solid))
@@
     (stroke (width 0) (type default))
   )
+  (wire (pts (xy 189.865 104.14) (xy 197.485 104.14))
+    (stroke (width 0) (type solid))
+  )
   (wire (pts (xy 419.1 48.26) (xy 419.1 52.07))
     (stroke (width 0) (type default))
@@
     (stroke (width 0) (type default))
   )
+  (wire (pts (xy 167.005 104.14) (xy 163.195 104.14))
+    (stroke (width 0) (type default))
+  )
   (wire (pts (xy 522.605 88.9) (xy 522.605 87.63))
     (stroke (width 0) (type default))
@@
     )
   )
+  (symbol (lib_name "PintryParts-Symbols:APA2107SECK_1") (lib_id "PintryParts-Symbols:APA2107SECK") (at 186.055 104.14 0) (mirror x) (unit 1)
+    (in_bom yes) (on_board yes) (dnp no) (fields_autoplaced)
+    (property "Reference" "D11" (at 184.4675 96.52 0)
+      (effects (font (size 1.27 1.27)))
+    )
+    (property "Value" "APA2107SECK" (at 184.4675 99.06 0)
+      (effects (font (size 1.27 1.27)))
+    )
+    (property "Footprint" "LED_SMD:LED_0603_1608Metric" (at 186.055 104.14 0)
+      (effects (font (size 1.27 1.27)) hide)
+    )
+    (property "Datasheet" "https://www.kingbrightusa.com/images/catalog/SPEC/APA2107SECK-J4-PRV.pdf" (at 185.42 113.03 0)
+      (effects (font (size 1.27 1.27)) hide)
+    )
+    (property "PartNumber" "APA2107SECK/J4-PRV" (at 185.42 112.395 0)
+      (effects (font (size 1.27 1.27)) hide)
+    )
+    (property "Manufacturer" "Kingbright" (at 184.15 113.03 0)
+      (effects (font (size 1.27 1.27)) hide)
+    )
+    (property "Part Number" "APA2107SECK/J4-PRV" (at 185.42 112.395 0)
+      (effects (font (size 1.27 1.27)) hide)
+    )
+    (pin "1")
+    (pin "2")
+    (instances
+      (project "gbc-cm4-aio"
+        (path "/4dda0f32-68f6-467e-9c4a-af7e2b8a8793"
+          (reference "D11") (unit 1)
+        )
+      )
+    )
+  )
   (symbol (lib_id "power:GND") (at 387.35 76.2 0) (unit 1)
     (in_bom yes) (on_board yes) (dnp no) (fields_autoplaced)
@@
     )
   )
+  (symbol (lib_id "power:GND") (at 163.195 104.14 270) (unit 1)
+    (in_bom yes) (on_board yes) (dnp no)
+    (property "Reference" "#PWR061" (at 156.845 104.14 0)
+      (effects (font (size 1.27 1.27)) hide)
+    )
+    (property "Value" "GND" (at 158.8008 104.267 0)
+      (effects (font (size 1.27 1.27)))
+    )
+    (property "Footprint" "" (at 163.195 104.14 0)
+      (effects (font (size 1.27 1.27)) hide)
+    )
+    (property "Datasheet" "" (at 163.195 104.14 0)
+      (effects (font (size 1.27 1.27)) hide)
+    )
+    (pin "1")
+    (instances
+      (project "gbc-cm4-aio"
+        (path "/4dda0f32-68f6-467e-9c4a-af7e2b8a8793"
+          (reference "#PWR061") (unit 1)
+        )
+      )
+      (project "MinCab"
+        (path "/bad99575-addb-4b0c-90c1-176ac3a4e3db"
+          (reference "#PWR04") (unit 1)
+        )
+      )
+    )
+  )
   (symbol (lib_id "power:+3.3V") (at 207.01 41.91 0) (mirror y) (unit 1)
     (in_bom yes) (on_board yes) (dnp no)
@@
     )
   )
+  (symbol (lib_id "power:+3.3V") (at 197.485 104.14 270) (mirror x) (unit 1)
+    (in_bom yes) (on_board yes) (dnp no) (fields_autoplaced)
+    (property "Reference" "#PWR058" (at 193.675 104.14 0)
+      (effects (font (size 1.27 1.27)) hide)
+    )
+    (property "Value" "+3.3V" (at 201.295 104.7749 90)
+      (effects (font (size 1.27 1.27)) (justify left))
+    )
+    (property "Footprint" "" (at 197.485 104.14 0)
+      (effects (font (size 1.27 1.27)) hide)
+    )
+    (property "Datasheet" "" (at 197.485 104.14 0)
+      (effects (font (size 1.27 1.27)) hide)
+    )
+    (pin "1")
+    (instances
+      (project "gbc-cm4-aio"
+        (path "/4dda0f32-68f6-467e-9c4a-af7e2b8a8793"
+          (reference "#PWR058") (unit 1)
+        )
+      )
+    )
+  )
   (symbol (lib_id "power:+3.3V") (at 402.59 118.11 0) (unit 1)
     (in_bom yes) (on_board yes) (dnp no)
@@
     )
   )
+  (symbol (lib_id "Device:R_US") (at 170.815 104.14 270) (mirror x) (unit 1)
+    (in_bom yes) (on_board yes) (dnp no)
+    (property "Reference" "R42" (at 172.8471 100.076 90)
+      (effects (font (size 1.27 1.27)) (justify left))
+    )
+    (property "Value" "1K" (at 172.7201 101.981 90)
+      (effects (font (size 1.27 1.27)) (justify left))
+    )
+    (property "Footprint" "Resistor_SMD:R_0603_1608Metric" (at 170.561 103.124 90)
+      (effects (font (size 1.27 1.27)) hide)
+    )
+    (property "Datasheet" "~" (at 170.815 104.14 0)
+      (effects (font (size 1.27 1.27)) hide)
+    )
+    (property "Tolerance" "1%" (at 168.275 100.076 90)
+      (effects (font (size 1.27 1.27)) (justify right))
+    )
+    (property "Size" "0603" (at 170.053 101.981 90)
+      (effects (font (size 1.27 1.27)) (justify right))
+    )
+    (pin "1")
+    (pin "2")
+    (instances
+      (project "gbc-cm4-aio"
+        (path "/4dda0f32-68f6-467e-9c4a-af7e2b8a8793"
+          (reference "R42") (unit 1)
+        )
+      )
+    )
+  )
   (symbol (lib_id "power:GND") (at 191.135 334.01 0) (unit 1)
     (in_bom yes) (on_board yes) (dnp no) (fields_autoplaced)
@@
       (effects (font (size 1.27 1.27)) (justify left))
     )
-    (property "Footprint" "Package_DFN_QFN:TDFN-14-1EP_3x3mm_P0.4mm_EP1.78x2.35mm" (at 288.29 81.28 0)
+    (property "Footprint" "Package_DFN_QFN:TDFN-8-1EP_2x2mm_P0.5mm_EP0.8x1.2mm" (at 288.29 81.28 0)
       (effects (font (size 1.27 1.27)) hide)
     )
-    (property "Datasheet" "https://datasheets.maximintegrated.com/en/ds/MAX17261.pdf" (at 288.29 76.2 0)
+    (property "Datasheet" "https://www.analog.com/media/en/technical-documentation/data-sheets/MAX17048-MAX17049.pdf" (at 288.29 76.2 0)
       (effects (font (size 1.27 1.27)) hide)
     )
