File: gbc-cm4-aio.kicad_sch (KiCad schematic)
At the start: 136 parts, among them J1 Conn_01x40, J2 AudioJack2_Ground_Switch, J4 DM3D-SF, J6 Conn_01x11, J7 Conn_01x02, P1 USB_C_Plug_USB2.0, Q1 2N7002E, Q1 AO4407C, SW1 SW_Push, SW2 BOOT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

Commit message: remove global_en, move boot to more accessible location
Parts:
- removed R41: 220R, Resistor_SMD:R_0603_1608Metric, symbol Device:R_Small_US
- removed SW5: GLOBAL_EN, Button_Switch_SMD:SW_SPST_B3U-1000P, symbol Switch:SW_Push
Other:
- note removed: "Low for <1ms to Power Up"
- moved on the sheet: R40, SW2

Commit message: led positioning improvement
Parts:
- removed U2: 74LVC1G07SE-7, Package_TO_SOT_SMD:SOT-353_SC-70-5, symbol CM4IO:74LVC1G07_copy
- D5: value APA2107SECK -> PWR
- D6: value APA2107SECK -> ACT
Connections:
- net PWR_LED: now also R7.2
Other:
- moved on the sheet: D5, R7

Commit message: move x button to avoid potential conflict with i2s
Connections:
- net BTN_X: now also Module1.40 (GPIO9); no longer Module1.27 (GPIO20)
Changed lines of the file:
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@@
 	)
 	(junction
-		(at 47.625 163.195)
-		(diameter 0)
-		(color 0 0 0 0)
-	)
-	(junction
 		(at 356.87 53.34)
 		(diameter 0)
@@
 	(wire
 		(pts
-			(xy 272.415 237.49) (xy 254.635 237.49)
-		)
-		(stroke
-			(width 0)
-			(type default)
-		)
-	)
-	(wire
-		(pts
 			(xy 254.635 252.73) (xy 272.415 252.73)
 		)
@@
 	(wire
 		(pts
+			(xy 193.675 252.73) (xy 175.895 252.73)
+		)
+		(stroke
+			(width 0)
+			(type default)
+		)
+	)
+	(wire
+		(pts
 			(xy 175.895 303.53) (xy 193.675 303.53)
 		)
@@
 	(wire
 		(pts
-			(xy 47.625 163.195) (xy 47.625 165.735)
-		)
-		(stroke
-			(width 0)
-			(type default)
-		)
-	)
-	(wire
-		(pts
 			(xy 254.635 265.43) (xy 272.415 265.43)
 		)
@@
 		)
 	)
-	(label "BTN_X"
-		(at 272.415 237.49 180)
-		(fields_autoplaced yes)
-		(effects
-			(font
-				(size 1.27 1.27)
-			)
-			(justify right bottom)
-		)
-	)
 	(label "DSI1_D1_N"
 		(at 127.635 306.07 180)
@@
 		)
 	)
+	(label "BTN_X"
+		(at 175.895 252.73 0)
+		(fields_autoplaced yes)
+		(effects
+			(font
+				(size 1.27 1.27)
+			)
+			(justify left bottom)
+		)
+	)

Commit message: Backlight driver improvement
Parts:
- removed C35: 1uF, Capacitor_SMD:C_0603_1608Metric, symbol Device:C
- removed D2: ${SIM.PARAMS}, Diode_SMD:D_1206_3216Metric, symbol Simulation_SPICE:DIODE
- removed R36: 10k, Resistor_SMD:R_0603_1608Metric, symbol Device:R
- removed R40: 220R, Resistor_SMD:R_0603_1608Metric, symbol Device:R_Small_US
- removed SW2: BOOT, Button_Switch_SMD:SW_SPST_B3U-1000P, symbol Switch:SW_Push
- removed U8: CAT4139, Package_TO_SOT_SMD:SOT-23-5_HandSoldering, symbol sft:CAT4139
- added SW4: SW_SPDT, Button_Switch_SMD:SW_SPDT_PCM12, symbol Switch:SW_SPDT
- added U2: FAN5333B, Package_TO_SOT_SMD:SOT-23-5_HandSoldering, symbol sft:CAT4139
- C34: value 220nF -> 1uF
- L3: value 22uH -> 6.8uH
- R12: value 1k -> 10k
Connections:
- net +2V8: no longer C32.1, C33.1, L3.1
- net +3V3: now also C32.1, C33.1, L3.1, U2.5 (VIN)
- net BL_EN: now also R9.1; no longer R9.2
- net BL_PWM: now also R11.1
- net DSI1_BL_A: now also C34.2, D1.1 (K)
- net DSI1_BL_K: now also U2.3 (FB); no longer R12.2
- net GND: now also C34.1, R12.1, SW4.3 (C), U2.2 (GND); no longer C34.2, R9.1
- net RPI_BOOT: now also SW4.2 (B)
- net at D1.2 (A), L3.2: now also U2.1 (SW)
- net at R11.2: now also R10.2, R12.2, R9.2, U2.4 (SHDN); no longer R12.1
Other:
- note removed: "Hold to boot from USB"
- moved on the sheet: +5V0, -5V0, 1V8, 2V8, 3V3, C27, C28, C29, C30, C31, C5, R4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

Commit message: cosmetics and optimizations
Parts:
- removed R9: 10k, Resistor_SMD:R_0603_1608Metric, symbol Device:R
Connections:
- net BL_EN: no longer names the net of Module1.30 (GPIO6)
Other:
- moved on the sheet: R10, R11
Changed lines of the file:
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@@
 	)
 	(junction
-		(at 38.1 169.545)
+		(at 38.1 161.29)
 		(diameter 0)
 		(color 0 0 0 0)
@@
 	)
 	(junction
-		(at 38.1 161.925)
-		(diameter 0)
-		(color 0 0 0 0)
-	)
-	(junction
 		(at 396.24 58.42)
 		(diameter 0)
@@
 	(wire
 		(pts
-			(xy 18.415 161.925) (xy 29.21 161.925)
-		)
-		(stroke
-			(width 0)
-			(type default)
-		)
-	)
-	(wire
-		(pts
 			(xy 118.745 121.92) (xy 118.745 125.095)
 		)
@@
 	(wire
 		(pts
-			(xy 38.1 169.545) (xy 36.83 169.545)
+			(xy 38.1 161.29) (xy 36.83 161.29)
 		)
 		(stroke
@@
 	(wire
 		(pts
-			(xy 36.83 161.925) (xy 38.1 161.925)
-		)
-		(stroke
-			(width 0)
-			(type default)
-		)
-	)
-	(wire
-		(pts
 			(xy 485.14 43.18) (xy 491.49 43.18)
 		)
@@
 	(wire
 		(pts
-			(xy 18.415 177.165) (xy 29.21 177.165)
+			(xy 18.415 168.91) (xy 29.21 168.91)
 		)
 		(stroke
@@
 	(wire
 		(pts
-			(xy 18.415 169.545) (xy 29.21 169.545)
+			(xy 18.415 161.29) (xy 29.21 161.29)
 		)
 		(stroke
@@
 	(wire
 		(pts
-			(xy 36.83 177.165) (xy 38.1 177.165)
+			(xy 36.83 168.91) (xy 38.1 168.91)
 		)
 		(stroke
@@
 	(wire
 		(pts
-			(xy 38.1 161.925) (xy 38.1 169.545)
-		)
-		(stroke
-			(width 0)
-			(type default)
-		)
-	)
-	(wire
-		(pts
 			(xy 254.635 300.99) (xy 277.495 300.99)
 		)
@@
 	(wire
 		(pts
-			(xy 38.1 177.165) (xy 38.1 169.545)
+			(xy 38.1 168.91) (xy 38.1 161.29)
 		)
 		(stroke
@@
 	(wire
 		(pts
-			(xy 38.1 161.925) (xy 38.1 154.94)
+			(xy 38.1 154.94) (xy 38.1 161.29)
 		)
 		(stroke
@@
 	(wire
 		(pts
-			(xy 175.895 240.03) (xy 193.675 240.03)
-		)
-		(stroke
-			(width 0)
-			(type default)
-		)
-	)
-	(wire
-		(pts
 			(xy 356.87 50.8) (xy 356.87 53.34)
 		)
@@
 		)
 	)
-	(label "BL_EN"
-		(at 18.415 161.925 0)
-		(fields_autoplaced yes)
-		(effects
-			(font
-				(size 1.27 1.27)
-			)
-			(justify left bottom)
-		)
-	)
 	(label "DSI1_CLK_P"
 		(at 127.635 316.23 180)
@@
 	)
 	(label "BL_PWM"
-		(at 18.415 177.165 0)
+		(at 18.415 168.91 0)
 		(fields_autoplaced yes)
 		(effects
@@
 		)
 	)
-	(label "BL_EN"
-		(at 175.895 240.03 0)
-		(fields_autoplaced yes)
-		(effects
-			(font
-				(size 1.27 1.27)
-			)
-			(justify left bottom)
-		)
-	)
 	(label "ACT_LED"
 		(at 272.415 229.87 180)
@@
 	)
 	(label "DSI1_PWM"
-		(at 18.415 169.545 0)
+		(at 18.415 161.29 0)
 		(fields_autoplaced yes)
 		(effects
@@
 	)
 	(symbol
-		(lib_id "Device:R")
-		(at 33.02 161.925 90)
-		(mirror x)
-		(unit 1)
-		(exclude_from_sim no)
-		(in_bom yes)
-		(on_board yes)
-		(dnp no)
-		(property "Reference" "R9"
-			(at 33.02 156.845 90)
-			(effects
-				(font
-					(size 1.27 1.27)
-				)
-			)
-		)
-		(property "Value" "10k"
-			(at 33.02 159.385 90)
-			(effects
-				(font
-					(size 1.27 1.27)
-				)
-			)
-		)
-		(property "Footprint" "Resistor_SMD:R_0603_1608Metric"
-			(at 33.02 160.147 90)
-			(effects
-				(font
-					(size 1.27 1.27)
-				)
-				(hide yes)
-			)
-		)
-		(property "Datasheet" "~"
-			(at 33.02 161.925 0)
-			(effects
-				(font
-					(size 1.27 1.27)
-				)
-				(hide yes)
-			)
-		)
-		(property "Description" ""
-			(at 33.02 161.925 0)
-			(effects
-				(font
-					(size 1.27 1.27)
-				)
-				(hide yes)
-			)
-		)
-		(pin "1"
-		)
-		(pin "2"
-		)
-		(instances
-			(project "gbc-cm4-aio"
-				(path "/4dda0f32-68f6-467e-9c4a-af7e2b8a8793"
-					(reference "R9")
-					(unit 1)
-				)
-			)
-		)
-	)
-	(symbol
 		(lib_id "Device:C")
 		(at 58.42 34.29 90)
@@
 	(symbol
 		(lib_id "Device:R")
-		(at 33.02 169.545 90)
+		(at 33.02 161.29 90)
 		(mirror x)
 		(unit 1)
@@
 		(dnp no)
 		(property "Reference" "R10"
-			(at 33.02 164.465 90)
+			(at 33.02 156.21 90)
 			(effects
 				(font
@@
 		)
 		(property "Value" "10k"
-			(at 33.02 167.005 90)
+			(at 33.02 158.75 90)
 			(effects
 				(font
@@
 		)
 		(property "Footprint" "Resistor_SMD:R_0603_1608Metric"
-			(at 33.02 167.767 90)
+			(at 33.02 159.512 90)
 			(effects
 				(font
@@
 		)
 		(property "Datasheet" "~"
-			(at 33.02 169.545 0)
+			(at 33.02 161.29 0)
 			(effects
 				(font
@@
 		)
 		(property "Description" ""
-			(at 33.02 169.545 0)
+			(at 33.02 161.29 0)
 			(effects
 				(font
@@
 				)
 				(justify left)
+				(hide yes)
 			)
 		)
@@
 	(symbol
 		(lib_id "Device:R")
-		(at 33.02 177.165 90)
+		(at 33.02 168.91 90)
 		(mirror x)
 		(unit 1)
@@
 		(dnp no)
 		(property "Reference" "R11"
-			(at 33.02 172.085 90)
+			(at 33.02 163.83 90)
 			(effects
 				(font
@@
 		)
 		(property "Value" "10k"
-			(at 33.02 174.625 90)
+			(at 33.02 166.37 90)
 			(effects
 				(font
@@
 		)
 		(property "Footprint" "Resistor_SMD:R_0603_1608Metric"
-			(at 33.02 175.387 90)
+			(at 33.02 167.132 90)
 			(effects
 				(font
@@
 		)
 		(property "Datasheet" "~"
-			(at 33.02 177.165 0)
+			(at 33.02 168.91 0)
 			(effects
 				(font
@@
 		)
 		(property "Description" ""
-			(at 33.02 177.165 0)
+			(at 33.02 168.91 0)
 			(effects
 				(font

Commit message: added battery gauge alert
Connections:
- net ALERT: now reaches Module1.30 (GPIO6)
- net ALERT: now also U4.5 (ALRT)
Changed lines of the file:
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@@
 	(wire
 		(pts
+			(xy 175.895 240.03) (xy 193.675 240.03)
+		)
+		(stroke
+			(width 0)
+			(type default)
+		)
+	)
+	(wire
+		(pts
 			(xy 520.065 203.2) (xy 520.065 205.74)
 		)
@@
 	(wire
 		(pts
+			(xy 308.61 45.72) (xy 298.45 45.72)
+		)
+		(stroke
+			(width 0)
+			(type default)
+		)
+	)
+	(wire
+		(pts
 			(xy 394.97 213.36) (xy 397.51 213.36)
 		)
@@
 		)
 	)
+	(label "ALERT"
+		(at 175.895 240.03 0)
+		(fields_autoplaced yes)
+		(effects
+			(font
+				(size 1.27 1.27)
+			)
+			(justify left bottom)
+		)
+	)
 	(label "NAV_UP"
 		(at 139.065 164.465 0)
@@
 		)
 	)
+	(label "ALERT"
+		(at 308.61 45.72 180)
+		(fields_autoplaced yes)
+		(effects
+			(font
+				(size 1.27 1.27)
+			)
+			(justify right bottom)
+		)
+	)
