File: PCBs/mainboard/gbc-cm4-aio.kicad_pcb (KiCad board)
At the start: 4 copper layers, 70.1 x 122.2 mm, 128 parts, among them J1 Conn_01x40, J2 AudioJack2_Ground_Switch, J4 DM3D-SF, J6 Conn_01x11, J7 Conn_01x02, P1 USB_C_Plug_USB2.0, Q1 AO4407C, Q3 2N7002E, SW1 SW_Push, SW3 SW_Push_Dual_x2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

Commit message: bump version number
Other:
- board text added: "GBC AIO v1.2"
- board text removed: "GBC AIO v1.1"
Changed lines of the file:
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@@
 		(tags "resistor")
 		(property "Reference" "R12"
-			(at -2.84 0.00125 270)
+			(at -2.84 0.00125 -90)
 			(layer "B.SilkS")
 			(effects
@@
 		)
 		(property "Value" "10k"
-			(at 0 -1.43 270)
+			(at 0 -1.43 -90)
 			(layer "B.Fab")
 			(effects
@@
 		)
 		(fp_text user "${REFERENCE}"
-			(at 0 0 270)
+			(at 0 0 -90)
 			(layer "B.Fab")
 			(effects
@@
 		(tags "capacitor")
 		(property "Reference" "C33"
-			(at 2.795 0 270)
+			(at 2.795 0 -90)
 			(layer "B.SilkS")
 			(effects
@@
 		)
 		(property "Value" "1uF"
-			(at 0 -1.43 270)
+			(at 0 -1.43 -90)
 			(layer "B.Fab")
 			(effects
@@
 		)
 		(fp_text user "${REFERENCE}"
-			(at 0 0 270)
+			(at 0 0 -90)
 			(layer "B.Fab")
 			(effects
@@
 		(tags "resistor")
 		(property "Reference" "R42"
-			(at 0.295 1.34 360)
+			(at 0.295 1.34 0)
 			(layer "B.SilkS")
 			(effects
@@
 		)
 		(property "Value" "1K"
-			(at 0 -1.43 360)
+			(at 0 -1.43 0)
 			(layer "B.Fab")
 			(effects
@@
 		)
 		(property "Size" "0603"
-			(at 0 0 360)
+			(at 0 0 0)
 			(layer "B.Fab")
 			(hide yes)
@@
 		)
 		(property "Tolerance" "1%"
-			(at 0 0 360)
+			(at 0 0 0)
 			(layer "B.Fab")
 			(hide yes)
@@
 		)
 		(fp_text user "${REFERENCE}"
-			(at 0 0 360)
+			(at 0 0 0)
 			(layer "B.Fab")
 			(effects
@@
 		)
 	)
-	(gr_text "GBC AIO v1.1"
+	(gr_text "GBC AIO v1.2"
 		(at 152.53 151.89 0)
 		(layer "B.SilkS")
@@
 		)
 	)
-	(gr_text "GBC AIO v1.1"
-		(at 149.5 252.17 -0)
+	(gr_text "GBC AIO v1.2"
+		(at 149.5 252.17 0)
 		(layer "F.SilkS")
 		(effects

Commit message: led backlight
Parts:
- added D12: WS2812B, LED_SMD:LED_WS2812B-2020_PLCC4_2.0x2.0mm, F.Cu at (143.0, 224.2)
- added D13: WS2812B, LED_SMD:LED_WS2812B-2020_PLCC4_2.0x2.0mm, F.Cu at (160.2, 224.3)
- added D14: WS2812B, LED_SMD:LED_WS2812B-2020_PLCC4_2.0x2.0mm, F.Cu at (160.3, 207.1)
- added D15: WS2812B, LED_SMD:LED_WS2812B-2020_PLCC4_2.0x2.0mm, F.Cu at (187.5, 224.3)
- added D16: WS2812B, LED_SMD:LED_WS2812B-2020_PLCC4_2.0x2.0mm, F.Cu at (194.0, 212.0)
- added D17: WS2812B, LED_SMD:LED_WS2812B-2020_PLCC4_2.0x2.0mm, F.Cu at (205.4, 218.7)
- added D18: WS2812B, LED_SMD:LED_WS2812B-2020_PLCC4_2.0x2.0mm, F.Cu at (181.1, 234.0)
- added D19: WS2812B, LED_SMD:LED_WS2812B-2020_PLCC4_2.0x2.0mm, F.Cu at (166.7, 234.2)
- added D2: WS2812B, LED_SMD:LED_WS2812B-2020_PLCC4_2.0x2.0mm, F.Cu at (143.0, 207.1)
- added D20: WS2812B, LED_SMD:LED_WS2812B-2020_PLCC4_2.0x2.0mm, F.Cu at (170.5, 240.9)
- added D21: WS2812B, LED_SMD:LED_WS2812B-2020_PLCC4_2.0x2.0mm, F.Cu at (177.6, 241.1)
- added U3: SN74LV1T34DCK, Package_TO_SOT_SMD:SOT-353_SC-70-5, B.Cu at (151.2, 197.3)
Connections:
- Module1 pad 58: unconnected-(Module1A-GPIO2-Pad58) -> /WS2812B
Routing:
- net Net-(D14-DOUT): track 0.00 -> 42.7 mm, vias 0 -> 2
- net Net-(D17-DOUT): track 0.00 -> 38.3 mm, vias 0 -> 2
- net /WS2812B: track 0.00 -> 26.4 mm, vias 0 -> 2
- net Net-(D12-DOUT): track 0.00 -> 17.6 mm, vias 0 -> 2
- net Net-(D15-DOUT): track 0.00 -> 17.0 mm, vias 0 -> 2
- net Net-(D12-DIN): track 0.00 -> 15.8 mm, vias 0 -> 2
- net Net-(D13-DOUT): track 0.00 -> 15.7 mm, vias 0 -> 2
- net Net-(D16-DOUT): track 0.00 -> 15.0 mm, vias 0 -> 2
- net Net-(D2-DIN): track 0.00 -> 14.4 mm, vias 0 -> 2
- net Net-(D18-DOUT): track 0.00 -> 13.4 mm, vias 0 -> 2
- net Net-(D19-DOUT): track 0.00 -> 10.2 mm, vias 0 -> 2
- net Net-(D20-DOUT): track 0.00 -> 5.66 mm
- net +5V: track 4.96 -> 6.59 mm, vias 45 -> 55
- net GND: vias 463 -> 462
