File: PCBs/mainboard/gbc-cm4-aio.kicad_pcb (KiCad board)
At the start: 4 copper layers, 70.1 x 122.2 mm, 125 parts, among them J1 Conn_01x40, J2 AudioJack2_Ground_Switch, J4 DM3D-SF, J6 Conn_01x11, J7 Conn_01x02, P1 USB_C_Plug_USB2.0, Q1 AO4407C, Q3 2N7002E, SW1 SW_Push, SW3 SW_Push_Dual_x2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

Commit message: minor optimizations
Parts:
- removed R14, R15: TBD, Resistor_SMD:R_0603_1608Metric
- removed R28, R29: 10K, Resistor_SMD:R_0603_1608Metric
- removed R30, R31: 2.2K 1%, Resistor_SMD:R_0603_1608Metric
- moved R2 6.84 mm to (178.3, 185.4), turned to 0 degrees
- moved R1 5.41 mm to (178.3, 184.0), turned to 0 degrees
- moved C17 5.15 mm to (156.8, 249.8), turned to -90 degrees
- moved C14 4.94 mm to (158.1, 249.8), turned to -90 degrees
- moved R42 4.35 mm to (150.6, 156.2)
- moved R32 3.74 mm to (194.1, 188.0)
- moved C3 3.74 mm to (187.0, 186.8)
- moved Q3 3.74 mm to (190.0, 186.6)
- moved R33 3.74 mm to (185.5, 186.8)
- moved D8 3.67 mm to (194.1, 186.6)
- moved U4 3.60 mm to (181.7, 185.3)
- moved C11 3.10 mm to (156.8, 252.8), turned to -90 degrees
- moved C40 1.79 mm to (160.1, 243.8)
- moved C13 1.59 mm to (158.1, 252.8), turned to -90 degrees
- moved R27 1.21 mm to (146.4, 238.0)
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Connections:
- Module1 pad 75: /SD_PWR_ON -> unconnected-(Module1A-SD_PWR_ON-Pad75)
- Module1 pad 80: /SCL0 -> unconnected-(Module1A-SCL0-Pad80)
- Module1 pad 82: /SDA0 -> unconnected-(Module1A-SDA0-Pad82)
- Module1 pad 99: /GLOBAL_EN -> unconnected-(Module1A-Global_EN-Pad99)
- U10 pad 5: Net-(U10-EN) -> /VIN
- U10 pad 6: Net-(U10-MODE) -> GND
- U9 pad 2: Net-(U9-VPCC) -> VBUS
Routing:
- net VBUS: track 171.4 -> 128.1 mm, vias 18 -> 16
- net /USB_OTG_ID: track 8.65 -> 0.00 mm, vias 2 -> 0
- net Net-(U9-VPCC): track 5.90 -> 0.00 mm
- net Net-(D8-A): track 16.1 -> 10.5 mm
- net GND: track 54.1 -> 48.8 mm, vias 464 -> 462
- net +BATT: track 81.3 -> 76.4 mm
- net Net-(U10-EN): track 4.64 -> 0.00 mm
- net /VBAT: track 25.2 -> 20.9 mm
- net Net-(D11-K): track 4.97 -> 9.17 mm, vias 1 -> 2
- net /VIN: track 88.5 -> 92.7 mm, vias 50 -> 51
- net Net-(D8-K): track 35.4 -> 32.0 mm, vias 0 -> 2
- net Net-(U10-MODE): track 2.91 -> 0.00 mm
- net /ALERT: track 10.8 -> 8.11 mm
- net Net-(U5-LDOO): track 2.97 -> 5.30 mm
- net /SDA1: track 31.1 -> 29.0 mm
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