File: PCBs/mainboard/gbc-cm4-aio.kicad_sch (KiCad schematic)
At the start: 126 parts, among them J1 Conn_01x40, J2 AudioJack2_Ground_Switch, J4 DM3D-SF, J6 Conn_01x11, J7 Conn_01x02, P1 USB_C_Plug_USB2.0, Q1 2N7002E, Q1 AO4407C, SW1 SW_Push, SW3 SW_Push_Dual_x2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

Commit message: led backlight
Parts:
- added D12, D13, D14, D15, D16, D17, D18, D19, D2, D20, D21: WS2812B, LED_SMD:LED_WS2812B-2020_PLCC4_2.0x2.0mm, symbol LED:WS2812B
- added U3: SN74LV1T34DCK, Package_TO_SOT_SMD:SOT-353_SC-70-5, symbol Logic_LevelTranslator:SN74LV1T34DCK
Connections:
- net +5V: now also D12.2 (VDD), D13.2 (VDD), D14.2 (VDD), D15.2 (VDD), D16.2 (VDD), D17.2 (VDD), D18.2 (VDD), D19.2 (VDD), D2.2 (VDD), D20.2 (VDD), D21.2 (VDD), U3.5 (VCC)
- net GND: now also D12.4 (VSS), D13.4 (VSS), D14.4 (VSS), D15.4 (VSS), D16.4 (VSS), D17.4 (VSS), D18.4 (VSS), D19.4 (VSS), D2.4 (VSS), D20.4 (VSS), D21.4 (VSS), U3.3 (GND)
- net WS2812B: now reaches Module1.58 (GPIO2)
- net WS2812B: now also U3.2 (A)
- new net: D2.1 (DIN), U3.4 (Y)
- new net: D12.1 (DIN), D2.3 (DOUT)
- new net: D19.3 (DOUT), D20.1 (DIN)
- new net: D20.3 (DOUT), D21.1 (DIN)
- new net: D18.3 (DOUT), D19.1 (DIN)
- new net: D16.3 (DOUT), D17.1 (DIN)
- new net: D17.3 (DOUT), D18.1 (DIN)
- new net: D14.3 (DOUT), D15.1 (DIN)
- new net: D15.3 (DOUT), D16.1 (DIN)
- new net: D12.3 (DOUT), D13.1 (DIN)
- new net: D13.3 (DOUT), D14.1 (DIN)
Other:
- note added: "RGB Backlight"
